File: designs/arena_10_of_10_v1r1/arena_10_of_10_v1r1.kicad_pcb (KiCad board)
At the start: 2 copper layers, 248.9 x 228.6 mm, 519 parts, among them J1 Cetus RJ45 Magjack, J10 Conn_01x05, J11 Conn_01x05, J12 Conn_01x05, J13 Conn_01x05, J14 Conn_01x05, J15 Conn_01x05, J16 Conn_01x05, J17 Conn_01x05, J18 Conn_01x05, J19 Conn_01x05, J2 Conn_01x02, J20 Conn_01x05, J21 Conn_01x05, J22 Conn_01x05, J23 Conn_01x05, J24 Conn_01x05, J25 Barrel_Jack, J26 Barrel_Jack, J27 Conn_Coaxial, J28 Conn_Coaxial, J29 Conn_Coaxial, J3 Conn_Coaxial, J4 Conn_Coaxial, J5 Conn_01x05, J6 Conn_01x05, J7 Conn_01x05, J8 Conn_01x05, J9 Conn_01x05, P1 NA, P10 NA, P2 NA, P3 NA, P4 NA, P5 NA, P6 NA, P7 NA, P8 NA, P9 NA, SW1 SW_SPDT, U1 Teensy4.1, U10 74LVC2G17, U100 74LVC1G125, U101 74LVC2G17, U102 SN74HCS08, U103 SN74HCS08, U104 74LVC1G125, U105 74LVC2G17, U106 SN74HCS08, U107 SN74HCS08, U108 74LVC1G125, U109 74LVC2G17, U11 74LVC2G17, U112 74LVC1G125, U113 74LVC2G17, U116 74LVC1G125, U117 74LVC2G17, U12 74LVC2G17, U120 74LVC1G125, U121 74LVC2G17, U124 74LVC1G125, U125 74LVC2G17, U13 74LVC2G17, U14 74LVC2G17, U15 74LVC2G17, U16 74LVC2G17, U17 74LVC2G17, U18 74LVC2G17, U19 74LVC2G17, U2 SN74LV1T34DBV, U20 74LVC2G17, U21 74LVC2G17, U22 74LVC2G17, U23 74LVC2G17, U24 74LVC2G17, U25 74LVC2G17, U26 74LVC2G17, U27 74LVC2G17, U28 74LVC2G17, U29 74LVC2G17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

Commit message: Work on layout and routing.
Parts:
- J25, J26: footprint arena_custom:DCJACK_2PIN_HIGHCURRENT -> arena_custom:DC-053D-20A
- moved C116 23.0 mm to (246.9, 89.4), turned to 90 degrees
- moved C133 18.3 mm to (256.6, 87.4), turned to 90 degrees
- moved R195 18.0 mm to (258.6, 87.4), turned to -90 degrees
- moved R196 16.5 mm to (254.5, 89.4), turned to -90 degrees
- moved U95 14.6 mm to (250.7, 94.1), turned to 90 degrees
- moved U100 13.7 mm to (257.6, 90.5), turned to 90 degrees
- moved J26 12.0 mm to (96.0, 75.6)
- moved J25 11.7 mm to (234.5, 75.5)
- moved R197 9.21 mm to (256.5, 94.2), turned to -90 degrees
- moved C117 8.75 mm to (257.5, 94.1), turned to 90 degrees
- moved R33 6.49 mm to (263.6, 225.5)
- moved R35 6.49 mm to (267.2, 225.5)
- moved C8 6.49 mm to (268.2, 225.5)
- moved R34 6.49 mm to (265.7, 225.4)
- moved U7 6.49 mm to (264.7, 228.5)
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Routing:
- net Net-(R190-Pad2): track 0.00 -> 1.97 mm
Other:
- outline, holes or cut-outs redrawn
- copper layers 2 -> 6

Commit message: More work on PCB layout & pre-routing board setup.
Parts:
- moved C118 5.90 mm to (274.0, 104.2)
- moved C119 5.90 mm to (269.1, 114.6)
- moved C134 5.90 mm to (276.0, 113.6)
- moved R198 5.90 mm to (276.0, 115.6)
- moved U104 5.90 mm to (272.9, 114.6)
- moved U105 5.90 mm to (266.0, 114.6)
- moved U98 5.90 mm to (269.3, 108.0)
- moved R199 5.90 mm to (274.1, 111.8)
- moved R200 5.90 mm to (269.1, 113.5)
- moved C33 4.20 mm to (305.3, 271.1)
- moved R82 4.20 mm to (306.3, 271.1)
- moved R83 4.20 mm to (304.3, 271.1)
- moved U33 4.20 mm to (305.3, 268.0)
- moved C34 4.17 mm to (301.6, 271.1)
- moved U34 4.17 mm to (301.6, 268.0)
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