File: designs/arena_10_of_10_v1r1/fan_out_by_2x.kicad_sch (KiCad schematic)
At the start: 4 parts, among them U16 74LVC2G17

Commit message: Added LCSC part numbers to Symbol Fields Table.
Parts:
- C16: LCSC Part # (none) -> C1525
- R48, R49: LCSC Part # (none) -> C25105
- U16: LCSC Part # (none) -> C7394037
Changed lines of the file:
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@@
+			)
+		)
+		(property "LCSC Part #" "C25105"
+			(at 100.33 43.18 90)
+			(effects
+				(font
+					(size 1.27 1.27)
+				)
+				(hide yes)
 			)
 		)
@@
 			)
 		)
+		(property "LCSC Part #" "C7394037"
+			(at 82.55 43.18 0)
+			(effects
+				(font
+					(size 1.27 1.27)
+				)
+				(hide yes)
+			)
+		)
 		(pin "3"
 		)
@@
 			)
 		)
+		(property "LCSC Part #" "C7394037"
+			(at 166.37 54.61 0)
+			(effects
+				(font
+					(size 1.27 1.27)
+				)
+				(hide yes)
+			)
+		)
 		(pin "3"
 		)
@@
 			)
 		)
+		(property "LCSC Part #" "C7394037"
+			(at 82.55 59.69 0)
+			(effects
+				(font
+					(size 1.27 1.27)
+				)
+				(hide yes)
+			)
+		)
 		(pin "3"
 		)
@@
 			)
 		)
+		(property "LCSC Part #" "C1525"
+			(at 151.13 49.53 0)
+			(effects
+				(font
+					(size 1.27 1.27)
+				)
+				(hide yes)
+			)
+		)
 		(pin "1"
 		)
@@
 			(effects
 				(font
+					(size 1.27 1.27)
+				)
+				(hide yes)
+			)
+		)
+		(property "LCSC Part #" "C25105"
+			(at 100.33 59.69 90)
+			(effects
+				(font
