File: designs/arena_10_of_10_v1r1/fan_out_by_5x.kicad_sch (KiCad schematic)
At the start: 11 parts, among them U4 74LVC2G17, U5 74LVC2G17, U6 74LVC2G17

Commit message: Added LCSC part numbers to Symbol Fields Table.
Parts:
- C4, C5, C6: LCSC Part # (none) -> C1525
- R28, R29, R30, R31, R32: LCSC Part # (none) -> C25105
- U4, U5, U6: LCSC Part # (none) -> C7394037
Changed lines of the file:
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@@
+			)
+		)
+		(property "LCSC Part #" "C7394037"
+			(at 73.66 55.88 0)
+			(effects
+				(font
+					(size 1.27 1.27)
+				)
+				(hide yes)
 			)
 		)
@@
 			)
 		)
+		(property "LCSC Part #" "C7394037"
+			(at 73.66 88.9 0)
+			(effects
+				(font
+					(size 1.27 1.27)
+				)
+				(hide yes)
+			)
+		)
 		(pin "3"
 		)
@@
 			)
 		)
+		(property "LCSC Part #" "C1525"
+			(at 229.87 48.26 0)
+			(effects
+				(font
+					(size 1.27 1.27)
+				)
+				(hide yes)
+			)
+		)
 		(pin "1"
 		)
@@
 		)
 		(property "Description" "Dual Buffer, Schmitt Triggered, Low-Voltage CMOS"
+			(at 205.74 53.34 0)
+			(effects
+				(font
+					(size 1.27 1.27)
+				)
+				(hide yes)
+			)
+		)
+		(property "LCSC Part #" "C7394037"
 			(at 205.74 53.34 0)
 			(effects
@@
 			)
 		)
+		(property "LCSC Part #" "C7394037"
+			(at 73.66 39.37 0)
+			(effects
+				(font
+					(size 1.27 1.27)
+				)
+				(hide yes)
+			)
+		)
 		(pin "3"
 		)
@@
 		(property "Description" "Resistor, small symbol"
 			(at 91.44 72.39 0)
+			(effects
+				(font
+					(size 1.27 1.27)
+				)
+				(hide yes)
+			)
+		)
+		(property "LCSC Part #" "C25105"
+			(at 91.44 72.39 90)
 			(effects
 				(font
@@
 			)
 		)
+		(property "LCSC Part #" "C7394037"
+			(at 73.66 72.39 0)
+			(effects
+				(font
+					(size 1.27 1.27)
+				)
+				(hide yes)
+			)
+		)
 		(pin "3"
 		)
@@
 			)
 		)
+		(property "LCSC Part #" "C25105"
+			(at 91.44 105.41 90)
+			(effects
+				(font
+					(size 1.27 1.27)
+				)
+				(hide yes)
+			)
+		)
 		(pin "2"
 		)
@@
 		(property "Description" "Resistor, small symbol"
 			(at 91.44 39.37 0)
+			(effects
+				(font
+					(size 1.27 1.27)
+				)
+				(hide yes)
+			)
+		)
+		(property "LCSC Part #" "C25105"
+			(at 91.44 39.37 90)
 			(effects
 				(font
@@
 			)
 		)
+		(property "LCSC Part #" "C7394037"
+			(at 73.66 121.92 0)
+			(effects
+				(font
+					(size 1.27 1.27)
+				)
+				(hide yes)
+			)
+		)
 		(pin "3"
 		)
@@
 			)
 		)
+		(property "LCSC Part #" "C1525"
+			(at 190.5 48.26 0)
+			(effects
+				(font
+					(size 1.27 1.27)
+				)
+				(hide yes)
+			)
+		)
 		(pin "1"
 		)
@@
 		(property "Description" "Resistor, small symbol"
 			(at 91.44 55.88 0)
+			(effects
+				(font
+					(size 1.27 1.27)
+				)
+				(hide yes)
+			)
+		)
+		(property "LCSC Part #" "C25105"
+			(at 91.44 55.88 90)
 			(effects
 				(font
@@
 			)
 		)
+		(property "LCSC Part #" "C25105"
+			(at 91.44 88.9 90)
+			(effects
+				(font
+					(size 1.27 1.27)
+				)
+				(hide yes)
+			)
+		)
 		(pin "2"
 		)
@@
 		)
 		(property "Description" "Dual Buffer, Schmitt Triggered, Low-Voltage CMOS"
+			(at 166.37 53.34 0)
+			(effects
+				(font
+					(size 1.27 1.27)
+				)
+				(hide yes)
+			)
+		)
+		(property "LCSC Part #" "C7394037"
 			(at 166.37 53.34 0)
 			(effects
@@
 			)
 		)
+		(property "LCSC Part #" "C7394037"
+			(at 73.66 105.41 0)
+			(effects
+				(font
+					(size 1.27 1.27)
+				)
+				(hide yes)
+			)
+		)
 		(pin "3"
 		)
@@
 		)
 		(property "Description" "Unpolarized capacitor"
+			(at 151.13 48.26 0)
+			(effects
+				(font
+					(size 1.27 1.27)
+				)
+				(hide yes)
+			)
+		)
+		(property "LCSC Part #" "C1525"
 			(at 151.13 48.26 0)
 			(effects
@@
 			(at 245.11 53.34 0)
 			(effects
+				(font
+					(size 1.27 1.27)
+				)
+				(hide yes)
+			)
+		)
+		(property "LCSC Part #" "C7394037"
+			(at 245.11 53.34 0)
+			(effects
