File: designs/arena_10_of_10_v1r1/miso_enable.kicad_sch (KiCad schematic)
At the start: 9 parts, among them U88 74LVC1G125, U89 SN74HCS08, U90 74LVC2G17

Commit message: Added LCSC part numbers to Symbol Fields Table.
Parts:
- C110, C111, C130: LCSC Part # (none) -> C1525
- R186, R188: LCSC Part # (none) -> C25105
- R187: LCSC Part # (none) -> C5948099
- U88: LCSC Part # (none) -> C7394030
- U89: LCSC Part # (none) -> C2868021
- U90: LCSC Part # (none) -> C7394037
Changed lines of the file:
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@@
+			)
+		)
+		(property "LCSC Part #" "C1525"
+			(at 186.69 49.53 0)
+			(effects
+				(font
+					(size 1.27 1.27)
+				)
+				(hide yes)
 			)
 		)
@@
 			)
 		)
+		(property "LCSC Part #" "C7394030"
+			(at 68.58 78.74 0)
+			(effects
+				(font
+					(size 1.27 1.27)
+				)
+				(hide yes)
+			)
+		)
 		(pin "2"
 		)
@@
 		)
 		(property "Description" "Resistor, small symbol"
+			(at 68.58 44.45 0)
+			(effects
+				(font
+					(size 1.27 1.27)
+				)
+				(hide yes)
+			)
+		)
+		(property "LCSC Part #" "C5948099"
 			(at 68.58 44.45 0)
 			(effects
@@
 			)
 		)
+		(property "LCSC Part #" "C7394037"
+			(at 246.38 81.28 0)
+			(effects
+				(font
+					(size 1.27 1.27)
+				)
+				(hide yes)
+			)
+		)
 		(pin "3"
 		)
@@
 			)
 		)
+		(property "LCSC Part #" "C2868021"
+			(at 115.57 46.99 90)
+			(effects
+				(font
+					(size 1.27 1.27)
+				)
+				(hide yes)
+			)
+		)
 		(pin "8"
 		)
@@
 			)
 		)
+		(property "LCSC Part #" "C25105"
+			(at 52.07 78.74 90)
+			(effects
+				(font
+					(size 1.27 1.27)
+				)
+				(hide yes)
+			)
+		)
 		(pin "2"
 		)
@@
 			)
 		)
+		(property "LCSC Part #" "C25105"
+			(at 90.17 78.74 90)
+			(effects
+				(font
+					(size 1.27 1.27)
+				)
+				(hide yes)
+			)
+		)
 		(pin "2"
 		)
@@
 		(property "Description" ""
 			(at 199.39 80.01 0)
+			(effects
+				(font
+					(size 1.27 1.27)
+				)
+				(hide yes)
+			)
+		)
+		(property "LCSC Part #" "C2868021"
+			(at 199.39 80.01 90)
 			(effects
 				(font
@@
 			)
 		)
+		(property "LCSC Part #" "C1525"
+			(at 224.79 49.53 0)
+			(effects
+				(font
+					(size 1.27 1.27)
+				)
+				(hide yes)
+			)
+		)
 		(pin "1"
 		)
@@
 			)
 		)
+		(property "LCSC Part #" "C2868021"
+			(at 115.57 59.69 90)
+			(effects
+				(font
+					(size 1.27 1.27)
+				)
+				(hide yes)
+			)
+		)
 		(pin "8"
 		)
@@
 		)
 		(property "Description" "Unpolarized capacitor"
+			(at 73.66 109.22 0)
+			(effects
+				(font
+					(size 1.27 1.27)
+				)
+				(hide yes)
+			)
+		)
+		(property "LCSC Part #" "C1525"
 			(at 73.66 109.22 0)
 			(effects
@@
 			)
 		)
+		(property "LCSC Part #" "C7394037"
+			(at 242.57 54.61 0)
+			(effects
+				(font
+					(size 1.27 1.27)
+				)
+				(hide yes)
+			)
+		)
 		(pin "3"
 		)
@@
 			)
 		)
+		(property "LCSC Part #" "C2868021"
+			(at 91.44 53.34 90)
+			(effects
+				(font
+					(size 1.27 1.27)
+				)
+				(hide yes)
+			)
+		)
 		(pin "8"
 		)
@@
 		)
 		(property "Description" "Dual Buffer, Schmitt Triggered, Low-Voltage CMOS"
+			(at 107.95 78.74 0)
+			(effects
+				(font
+					(size 1.27 1.27)
+				)
+				(hide yes)
+			)
+		)
+		(property "LCSC Part #" "C7394037"
 			(at 107.95 78.74 0)
 			(effects
@@
 			(at 201.93 54.61 0)
 			(effects
+				(font
+					(size 1.27 1.27)
+				)
+				(hide yes)
+			)
+		)
+		(property "LCSC Part #" "C2868021"
+			(at 201.93 54.61 0)
+			(effects

Commit message: Added silkscreens.  Added required FT Rotations/Offsets for JLCPCB.
Parts:
- U88: LCSC Part # C7394030 -> C7394017
Changed lines of the file:
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@@
 			)
 		)
-		(property "LCSC Part #" "C7394030"
+		(property "LCSC Part #" "C7394017"
 			(at 68.58 78.74 0)
 			(effects
