File: arena_10-10/arena_top_10-10/panel_column.kicad_sch (KiCad schematic)
At the start: 4 parts, among them J5 Conn_01x05, J6 Conn_01x05, P1 NA

Commit message: fix connector, bump to v1.1.8
Parts:
- J5, J6: LCSC Part # C50950 -> C492404
Changed lines of the file:
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@@
 	(title_block
 		(title "G6 10-10 Arena Top")
-		(date "2026-05-26")
-		(rev "v1.1.0")
+		(date "2026-06-10")
+		(rev "v1.1.8")
 		(company "IORodeo for Reiser Lab @ Janelia | HHMI")
 	)
@@
 			)
 		)
-		(property "LCSC Part #" "C50950"
+		(property "LCSC Part #" "C492404"
 			(at 161.29 69.85 0)
 			(hide yes)
@@
 			)
 		)
-		(property "LCSC Part #" "C50950"
+		(property "LCSC Part #" "C492404"
 			(at 161.29 85.09 0)
 			(hide yes)
