File: arena_10-14/arena_10-14.kicad_pcb (KiCad board)
At the start: 6 copper layers, 330 x 240.1 mm, 623 parts, among them J1 Cetus RJ45 Magjack, J10 Conn_01x05, J11 Conn_01x05, J12 Conn_01x05, J13 Conn_01x05, J14 Conn_01x05, J15 Conn_01x05, J16 Conn_01x05, J17 Conn_01x05, J18 Conn_01x05, J19 Conn_01x05, J2 Qwiic, J20 Conn_01x05, J21 Conn_01x05, J22 Conn_01x05, J23 Conn_01x05, J24 Conn_01x05, J25 Conn_01x05, J26 Conn_01x05, J27 Barrel_Jack, J28 Barrel_Jack, J29 Conn_Coaxial, J3 Conn_01x02, J30 Conn_Coaxial, J31 Conn_Coaxial, J32 Conn_01x05, J33 Conn_01x05, J34 Conn_01x05, J35 Conn_01x05, J4 Conn_01x02, J5 Conn_Coaxial, J6 Conn_Coaxial, J7 Conn_01x05, J8 Conn_01x05, J9 Conn_01x05, P1 NA, P10 NA, P11 NA, P12 NA, P2 NA, P3 NA, P4 NA, P5 NA, P6 NA, P7 NA, P8 NA, P9 NA, SW1 SW_SPDT, U1 Teensy4.1, U10 74LVC2G17, U100 74LVC1G125, U101 SN74HCS08, U102 74LVC2G17, U103 74LVC1G125, U104 SN74HCS08, U105 74LVC2G17, U106 74LVC1G125, U107 SN74HCS08, U108 74LVC2G17, U109 74LVC1G125, U11 74LVC2G17, U110 SN74HCS08, U111 74LVC2G17, U112 74LVC1G125, U113 SN74HCS08, U114 74LVC2G17, U115 74LVC1G125, U116 SN74HCS08, U117 74LVC2G17, U118 74LVC2G17, U119 74LVC2G17, U12 74LVC2G17, U120 74LVC2G17, U121 74LVC2G17, U122 74LVC1G125, U123 SN74HCS08, U124 74LVC2G17, U125 74LVC1G125, U126 SN74HCS08, U127 74LVC2G17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

Commit message: edge cuts
Other:
- board size 330 x 240.1 mm -> 299.8 x 238.5 mm
Changed lines of the file:
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@@
 		(layer "B.SilkS")
 	)
-	(gr_curve
-		(pts
-			(xy 31 108) (xy 31 99.2) (xy 44.6 98.8) (xy 51 98.8)
+	(gr_line
+		(start 54.83 315.4)
+		(end 54.88 79.53)
+		(stroke
+			(width 0.3)
+			(type default)
 		)
+		(layer "Edge.Cuts")
+	)
+	(gr_line
+		(start 54.88 79.53)
+		(end 354.44 80.14)
+		(stroke
+			(width 0.3)
+			(type default)
+		)
+		(layer "Edge.Cuts")
+	)
+	(gr_line
+		(start 139.087226 313.917354)
+		(end 54.83 315.4)
+		(stroke
+			(width 0.3)
+			(type default)
+		)
+		(layer "Edge.Cuts")
+	)
+	(gr_arc
+		(start 139.087226 313.917354)
+		(mid 199.363384 148.555976)
+		(end 247.5 317.85)
 		(stroke
 			(width 0.3)
@@
 	)
 	(gr_line
-		(start 31 207)
-		(end 31 108)
-		(stroke
-			(width 0.3)
-			(type solid)
-		)
-		(layer "Edge.Cuts")
-	)
-	(gr_curve
-		(pts
-			(xy 31 261) (xy 31 253.4) (xy 41 250.8) (xy 41 241)
-		)
-		(stroke
-			(width 0.3)
-			(type solid)
-		)
-		(layer "Edge.Cuts")
-	)
-	(gr_curve
-		(pts
-			(xy 41 241) (xy 41 227.4) (xy 31 214.6) (xy 31 207)
-		)
-		(stroke
-			(width 0.3)
-			(type solid)
-		)
-		(layer "Edge.Cuts")
-	)
-	(gr_curve
-		(pts
-			(xy 51 98.8) (xy 57.4 98.8) (xy 103.2 101.6) (xy 121.8 85.8)
-		)
-		(stroke
-			(width 0.3)
-			(type default)
-		)
-		(layer "Edge.Cuts")
-	)
-	(gr_curve
-		(pts
-			(xy 85.2 303) (xy 88.6 308.4) (xy 83.6 311) (xy 78.8 311)
-		)
-		(stroke
-			(width 0.3)
-			(type solid)
-		)
-		(layer "Edge.Cuts")
-	)
-	(gr_arc
-		(start 107.878 311.13)
-		(mid 73.961239 295.706023)
-		(end 60.078 261.13)
-		(stroke
-			(width 0.3)
-			(type solid)
-		)
-		(layer "Edge.Cuts")
-	)
-	(gr_arc
-		(start 114.278 303.13)
-		(mid 225.078 114.130001)
-		(end 335.878 303.13)
-		(stroke
-			(width 0.3)
-			(type solid)
-		)
-		(layer "Edge.Cuts")
-	)
-	(gr_curve
-		(pts
-			(xy 121.8 85.8) (xy 140.4 70) (xy 145.8 71) (xy 153 71)
-		)
-		(stroke
-			(width 0.3)
-			(type solid)
-		)
-		(layer "Edge.Cuts")
-	)
-	(gr_line
-		(start 153 71)
-		(end 351 71)
-		(stroke
-			(width 0.3)
-			(type solid)
-		)
-		(layer "Edge.Cuts")
-	)
-	(gr_curve
-		(pts
-			(xy 306.8 303) (xy 303.6 308.4) (xy 308.4 311) (xy 313.2 311)
-		)
-		(stroke
-			(width 0.3)
-			(type default)
-		)
-		(layer "Edge.Cuts")
-	)
-	(gr_arc
-		(start 351 71)
-		(mid 358.071068 73.928932)
-		(end 361 81)
-		(stroke
-			(width 0.3)
-			(type default)
-		)
-		(layer "Edge.Cuts")
-	)
-	(gr_curve
-		(pts
-			(xy 351 241) (xy 351 227.4) (xy 361 214.6) (xy 361 207)
-		)
-		(stroke
-			(width 0.3)
-			(type solid)
-		)
-		(layer "Edge.Cuts")
-	)
-	(gr_arc
-		(start 353.8 85.414213)
-		(mid 353.8 84)
-		(end 355.214213 84)
+		(start 354.44 80.14)
+		(end 354.63 317.98)
 		(stroke
 			(width 0.3)
@@
 	)
 	(gr_line
-		(start 353.8 91.385787)
-		(end 353.8 85.414213)
+		(start 354.63 317.98)
+		(end 247.5 317.85)
 		(stroke
 			(width 0.3)
@@
 		)
 		(layer "Edge.Cuts")
-	)
-	(gr_arc
-		(start 355.214213 92.8)
-		(mid 353.8 92.8)
-		(end 353.8 91.385787)
-		(stroke
-			(width 0.3)
-			(type default)
-		)
-		(layer "Edge.Cuts")
-	)
-	(gr_line
-		(start 358 84)
-		(end 355.214213 84)
-		(stroke
-			(width 0.3)
-			(type default)
-		)
-		(layer "Edge.Cuts")
-	)
-	(gr_line
-		(start 358 92.8)
-		(end 355.214213 92.8)
-		(stroke
-			(width 0.3)
-			(type default)
-		)
-		(layer "Edge.Cuts")
-	)
-	(gr_arc
-		(start 358 92.8)
-		(mid 360.12132 93.67868)
-		(end 361 95.8)
-		(stroke
-			(width 0.3)
-			(type default)
-		)
-		(layer "Edge.Cuts")
-	)
-	(gr_arc
-		(start 361 81)
-		(mid 360.12132 83.12132)
-		(end 358 84)
-		(stroke
-			(width 0.3)
-			(type default)
-		)
-		(layer "Edge.Cuts")
-	)
-	(gr_line
-		(start 361 95.8)
-		(end 361 207)
-		(stroke
-			(width 0.3)
-			(type solid)
-		)
-		(layer "Edge.Cuts")
-	)
-	(gr_arc
-		(start 361 261)
-		(mid 346.355339 296.355339)
-		(end 313.2 311)
-		(stroke
-			(width 0.3)
-			(type solid)
-		)
-		(layer "Edge.Cuts")
-	)
-	(gr_curve
-		(pts
-			(xy 361 261) (xy 361 253.4) (xy 351 250.8) (xy 351 241)
-		)
-		(stroke
-			(width 0.3)
-			(type solid)
-		)
-		(layer "Edge.Cuts")
