File: arena_10-14/arena_10-14.kicad_pcb (KiCad board)
At the start: 6 copper layers, 270 x 208.3 mm, 566 parts, among them J1 Cetus RJ45 Magjack, J10 Conn_01x05, J11 Conn_01x05, J12 Conn_01x05, J13 Conn_01x05, J14 Conn_01x05, J15 Conn_01x05, J16 Conn_01x05, J17 Conn_01x05, J18 Conn_01x05, J19 Conn_01x05, J2 Qwiic, J20 Conn_01x05, J21 Conn_01x05, J22 Conn_01x05, J23 Conn_01x05, J24 Conn_01x05, J25 Conn_Coaxial, J26 Conn_Coaxial, J27 Barrel_Jack, J29 Conn_Coaxial, J3 Conn_01x02, J30 Conn_Coaxial, J31 Conn_Coaxial, J32 Conn_01x05, J33 Conn_01x05, J34 Conn_Coaxial, J35 JST PH, J4 Conn_01x02, J5 XT30, J6 Conn_Coaxial, J7 Conn_01x05, J8 Conn_01x05, J9 Conn_01x05, P1 NA, P10 NA, P2 NA, P3 NA, P4 NA, P5 NA, P6 NA, P7 NA, P8 NA, P9 NA, SW1 SW_SPDT, U1 Teensy4.1, U10 74LVC2G17, U100 74LVC1G125, U101 SN74HCS08, U102 74LVC2G17, U103 74LVC1G125, U104 SN74HCS08, U105 74LVC2G17, U106 74LVC1G125, U107 SN74HCS08, U108 74LVC2G17, U109 74LVC1G125, U11 74LVC2G17, U110 SN74HCS08, U111 74LVC2G17, U112 74LVC1G125, U113 SN74HCS08, U114 74LVC2G17, U12 74LVC2G17, U122 74LVC1G125, U123 SN74HCS08, U124 74LVC2G17, U128 74LVC2G17, U129 74LVC2G17, U13 74LVC2G17, U130 74LVC2G17, U131 74LVC2G17, U14 74LVC2G17, U15 74LVC2G17, U16 74LVC2G17, U17 74LVC2G17, U18 74LVC2G17, U19 74LVC2G17, U20 74LVC2G17, U21 74LVC2G17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

Commit message: H7 cleanup
Routing:
- net /Fan Out/PAN.CS_16_P5: track 223.9 -> 221.7 mm
- net /Fan Out/PAN.CS_17_P5: track 214.9 -> 213.2 mm
- net /Fan Out/PAN.CS_19_P5: track 228.0 -> 226.3 mm
- net /Fan Out/PAN.CS_18_P5: track 221.4 -> 220.0 mm
