File: arena_10-14/DIO.kicad_sch (KiCad schematic)
At the start: 2 parts, among them J6 Conn_Coaxial, U3 SN74LVC1T45DBV

Commit message: first draft
Parts:
- added C89, C90: 0.1uF, Capacitor_SMD:C_0402_1005Metric, symbol Device:C
Connections:
- net +3.3V: now also C90.1
- net +5V: now also C89.1
- net GND: now also C89.2, C90.2

Commit message: first moat
Parts:
- J6: footprint BNC:BNC -> BNC:BNC_HenryTech_HL-BNC_KHDA; LCSC Part # C2837587 -> C19712152
Changed lines of the file:
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@@
 			)
 		)
-		(property "Footprint" "BNC:BNC"
+		(property "Footprint" "BNC:BNC_HenryTech_HL-BNC_KHDA"
 			(at 137.16 85.09 0)
 			(hide yes)
@@
 			)
 		)
-		(property "LCSC Part #" "C2837587"
+		(property "LCSC Part #" "C19712152"
 			(at 137.16 85.09 0)
 			(hide yes)

Commit message: fix BNC export
Parts:
- J6: FT Rotation Offset 180 -> (none)
Changed lines of the file:
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@@
-			)
-		)
-		(property "FT Rotation Offset" "180"
-			(at 137.16 85.09 0)
-			(hide yes)
-			(show_name no)
-			(do_not_autoplace no)
-			(effects
-				(font
-					(size 1.27 1.27)
-				)
 			)
 		)
