File: arena_10-14/analog.kicad_sch (KiCad schematic)
At the start: 38 parts, among them J29 Conn_Coaxial, J30 Conn_Coaxial, J31 Conn_Coaxial, U83 OPA2277, U84 REF102AU, U85 MCP4725xxx-xCH, U86 OPA2277, U87 OPA2277

Commit message: rotate teensy
Parts:
- R189, R190: value 20k -> 10k; LCSC Part # C705630 -> C190095
- R191, R192: value 10k -> 20k; LCSC Part # C190095 -> C705630
Changed lines of the file:
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@@
 			)
 		)
-		(property "Value" "20k"
+		(property "Value" "10k"
 			(at 101.854 137.16 0)
 			(show_name no)
@@
 			)
 		)
-		(property "LCSC Part #" "C705630 "
+		(property "LCSC Part #" "C190095"
 			(at 97.79 135.89 0)
 			(hide yes)
@@
 			)
 		)
-		(property "Value" "20k"
+		(property "Value" "10k"
 			(at 105.664 105.41 0)
 			(show_name no)
@@
 			)
 		)
-		(property "LCSC Part #" "C705630 "
+		(property "LCSC Part #" "C190095"
 			(at 101.6 104.14 0)
 			(hide yes)
@@
 			)
 		)
-		(property "Value" "10k"
+		(property "Value" "20k"
 			(at 107.442 129.032 90)
 			(show_name no)
@@
 			)
 		)
-		(property "LCSC Part #" "C190095 "
+		(property "LCSC Part #" "C705630"
 			(at 104.14 130.81 90)
 			(hide yes)
@@
 			)
 		)
-		(property "Value" "10k"
+		(property "Value" "20k"
 			(at 111.252 97.282 90)
 			(show_name no)
@@
 			)
 		)
-		(property "LCSC Part #" "C190095 "
+		(property "LCSC Part #" "C705630"
 			(at 107.95 99.06 90)
 			(hide yes)

Commit message: first moat
Parts:
- J29, J30, J31: footprint BNC:BNC -> BNC:BNC_HenryTech_HL-BNC_KHDA; LCSC Part # C2837587 -> C19712152
Changed lines of the file:
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@@
 			)
 		)
-		(property "Footprint" "BNC:BNC"
+		(property "Footprint" "BNC:BNC_HenryTech_HL-BNC_KHDA"
 			(at 176.53 128.27 0)
 			(hide yes)
@@
 			)
 		)
-		(property "LCSC Part #" "C2837587"
+		(property "LCSC Part #" "C19712152"
 			(at 176.53 128.27 0)
 			(hide yes)
@@
 			)
 		)
-		(property "Footprint" "BNC:BNC"
+		(property "Footprint" "BNC:BNC_HenryTech_HL-BNC_KHDA"
 			(at 180.34 96.52 0)
 			(hide yes)
@@
 			)
 		)
-		(property "LCSC Part #" "C2837587"
+		(property "LCSC Part #" "C19712152"
 			(at 180.34 96.52 0)
 			(hide yes)
@@
 			)
 		)
-		(property "Footprint" "BNC:BNC"
+		(property "Footprint" "BNC:BNC_HenryTech_HL-BNC_KHDA"
 			(at 99.06 43.18 0)
 			(hide yes)
@@
 			)
 		)
-		(property "LCSC Part #" "C2837587"
+		(property "LCSC Part #" "C19712152"
 			(at 99.06 43.18 0)
 			(hide yes)

Commit message: better 15V GND
Parts:
- added TP3: 10V REF, TestPoint:TestPoint_Pad_D1.5mm, symbol Connector:TestPoint
- added TP4: +15V, TestPoint:TestPoint_Pad_D1.5mm, symbol Connector:TestPoint
- added TP5: -15V, TestPoint:TestPoint_Pad_D1.5mm, symbol Connector:TestPoint
- added TP6: AI2, TestPoint:TestPoint_Pad_D1.5mm, symbol Connector:TestPoint
- added TP7: AI1, TestPoint:TestPoint_Pad_D1.5mm, symbol Connector:TestPoint
Connections:
- net +15V: now also TP4.1
- net -15V: now also TP5.1
- net 10V_REF: now also TP3.1
- net A0_5V renamed A0_10V
- net A0_10V: now also TP7.1
- net A1_5V renamed A1_10V
- net A1_10V: now also TP6.1

Commit message: H7 cleanup
Parts:
- R193, R196: LCSC Part # C190095 -> C190095
- TP3, TP4, TP5, TP6, TP7: now not fitted; now left out of the parts list
Changed lines of the file:
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@@
 		(body_style 1)
 		(exclude_from_sim no)
-		(in_bom yes)
+		(in_bom no)
 		(on_board yes)
-		(in_pos_files yes)
-		(dnp no)
+		(in_pos_files no)
+		(dnp yes)
 		(fields_autoplaced yes)
 		(property "Reference" "TP3"
@@
 		(body_style 1)
 		(exclude_from_sim no)
-		(in_bom yes)
+		(in_bom no)
 		(on_board yes)
-		(in_pos_files yes)
-		(dnp no)
+		(in_pos_files no)
+		(dnp yes)
 		(fields_autoplaced yes)
 		(property "Reference" "TP4"
@@
 		(body_style 1)
 		(exclude_from_sim no)
-		(in_bom yes)
+		(in_bom no)
 		(on_board yes)
-		(in_pos_files yes)
-		(dnp no)
+		(in_pos_files no)
+		(dnp yes)
 		(fields_autoplaced yes)
 		(property "Reference" "TP6"
@@
 			)
 		)
-		(property "LCSC Part #" "C190095 "
+		(property "LCSC Part #" "C190095"
 			(at 163.83 96.52 90)
 			(hide yes)
@@
 		(body_style 1)
 		(exclude_from_sim no)
-		(in_bom yes)
+		(in_bom no)
 		(on_board yes)
-		(in_pos_files yes)
-		(dnp no)
+		(in_pos_files no)
+		(dnp yes)
 		(fields_autoplaced yes)
 		(property "Reference" "TP5"
@@
 			)
 		)
-		(property "LCSC Part #" "C190095 "
+		(property "LCSC Part #" "C190095"
 			(at 130.81 123.19 0)
 			(hide yes)
@@
 		(body_style 1)
 		(exclude_from_sim no)
-		(in_bom yes)
+		(in_bom no)
 		(on_board yes)
-		(in_pos_files yes)
-		(dnp no)
+		(in_pos_files no)
+		(dnp yes)
 		(fields_autoplaced yes)
 		(property "Reference" "TP7"

Commit message: fix BNC export
Parts:
- J29, J30, J31: FT Rotation Offset 180 -> (none)
Changed lines of the file:
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@@
 			)
 		)
-		(property "FT Rotation Offset" "180"
-			(at 176.53 128.27 0)
-			(hide yes)
-			(show_name no)
-			(do_not_autoplace no)
-			(effects
-				(font
-					(size 1.27 1.27)
-				)
-			)
-		)
 		(pin "2"
 		)
@@
 			)
 		)
-		(property "FT Rotation Offset" "180"
-			(at 180.34 96.52 0)
-			(hide yes)
-			(show_name no)
-			(do_not_autoplace no)
-			(effects
-				(font
-					(size 1.27 1.27)
-				)
-			)
-		)
 		(pin "2"
 		)
@@
 			(at 99.06 43.18 0)
 			(hide yes)
-			(show_name no)
-			(do_not_autoplace no)
-			(effects
-				(font
-					(size 1.27 1.27)
-				)
-			)
-		)
-		(property "FT Rotation Offset" "180"
-			(at 99.06 43.18 0)
-			(hide yes)

Commit message: Link DIO 3 & 4 DIR, place connectors
Parts:
- R194, R195: LCSC Part # C190095 -> C190095
Changed lines of the file:
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@@
 			)
 		)
-		(property "LCSC Part #" "C190095 "
+		(property "LCSC Part #" "C190095"
 			(at 160.02 128.27 90)
 			(hide yes)
@@
 			)
 		)
-		(property "LCSC Part #" "C190095 "
+		(property "LCSC Part #" "C190095"
 			(at 134.62 91.44 0)
 			(hide yes)
