File: arena_10-14/fan_out.kicad_sch (KiCad schematic)
At the start: 0 parts

Commit message: feat: reduce 10-14 arena to 10 panel columns and add digital IO channels
Schematic
- Remove panel columns P11 and P12; the Panels sheet now holds P1..P10.
- Re-split the SPI banks for 10 panels: B0 serves P1-P5, B1 serves
  P6-P10 (CIPO enables, SCK/COPI/EINT fan-out).
- Re-pair the chip selects: CS_00..19 each fan out to (Pn, Pn+5), and
  the CS_20..23 fan-out sheets are gone.
- The shared SCK/COPI/EINT dual buffers now drive P1/P2, P3/P4, P6/P7
  and P8/P9. The buffers for P5 and P10 each drive a single panel.
- Move the Teensy digital IO channel (SN74LVC1T45 level shifter and BNC
  connector) into a new DIO.kicad_sch sub-sheet and instance it four
  times (Digital IO 01..04).

PCB
- Update from the schematic: the P11/P12 columns and their parts are
  removed (623 -> 547 footprints, no P11/P12 nets left). The freed
  references U78-U80, J25, J26 and J34 now belong to the digital IO
  channels.
- Most of the old 12-panel routing is removed (4471 -> 1393
  tracks/vias).

Placement scripts (assets/placement/)
- 01, 02: end each footprint block at its own closing paren. The last
  footprint in the file used to extend to the end of the file, so 02
  added an angle to every via and KiCad refused to open the board
  ("Expecting ')'").
- 03: replicate to P1..P10 only and ignore CIPO-enable sheets beyond
  P10. Read the B0/B1 bank of the PAN and TNY nets from the board
  instead of hardcoding P1-P6 / P7-P12. Same footprint-block fix.
- 05: read each CS group's panel pair and midpoint anchor from the
  fan-out sheet names instead of hardcoding P(4+j), and stop if a
  midpoint is not a populated connector. Same footprint-block fix (05
  rewrites footprints, so it could corrupt vias the same way 02 did).

Known gaps, to follow up
- 05 stops on the new CS pairing: the P1/P6 midpoint is P3.5, so an
  anchor for each group still has to be chosen.
- 02 and 03 still pair the shared buffers as P1/P2, P3/P4, P5/P6,
  P7/P8, P9/P10, anchored on the even connector. With the new B1
  p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
Other:
- sheet CIPO B0 Enable for P6 renamed CIPO B1 Enable for P6
- sheet COPI B1 fan out to P7-P12 renamed COPI B1 fan out to P6-P10
- sheet CS_00 fan out to P1, P7 renamed CS_00 fan out to P1, P6
- sheet CS_01 fan out to P1, P7 renamed CS_01 fan out to P1, P6
- sheet CS_02 fan out to P1, P7 renamed CS_02 fan out to P1, P6
- sheet CS_03 fan out to P1, P7 renamed CS_03 fan out to P1, P6
- sheet CS_04 fan out to P2, P8 renamed CS_04 fan out to P2, P7
- sheet CS_05 fan out to P2, P8 renamed CS_05 fan out to P2, P7
- sheet CS_06 fan out to P2, P8 renamed CS_06 fan out to P2, P7
- sheet CS_07 fan out to  P2, P8 renamed CS_07 fan out to  P2, P7
- sheet CS_08 fan out to  P3, P9 renamed CS_08 fan out to  P3, P8
- sheet CS_09 fan out to P3, P9 renamed CS_09 fan out to P3, P8
- sheet CS_10 fan out to P3, P9 renamed CS_10 fan out to P3, P8
- sheet CS_11 fan out to P3, P9 renamed CS_11 fan out to P3, P8
- sheet CS_12 fan out to P4, P10 renamed CS_12 fan out to P4, P9
- sheet CS_13 fan out to P4, P10 renamed CS_13 fan out to P4, P9
- sheet CS_14 fan out to P4, P10 renamed CS_14 fan out to P4, P9
- sheet CS_15 fan out to P4, P10 renamed CS_15 fan out to P4, P9
- sheet CS_16 fan out to P5, P11 renamed CS_16 fan out to P5, P10
- sheet CS_17 fan out to P5, P11 renamed CS_17 fan out to P5, P10
- sheet CS_18 fan out to P5, P11 renamed CS_18 fan out to P5, P10
- sheet CS_19 fan out to P5, P11 renamed CS_19 fan out to P5, P10
- sheet EINT fan out to P1-P6 renamed EINT fan out to P1-P5
- sheet EINT fan out to P7-P12 renamed EINT fan out to P6-P10
- sheet SCK B1 fan out to P7-P12 renamed SCK B1 fan out to P6-P10
- removed sheet CIPO B1 Enable for P11
- removed sheet CIPO B1 Enable for P12
- removed sheet CS_20 fan out to P6, P12
- removed sheet CS_21 fan out to P6, P12
- removed sheet CS_22 fan out to P6, P12
- removed sheet CS_23 fan out to P6, P12
- note added: "Chip Select P1-P10"
- note removed: "Chip Select P1-P12"

Commit message: first draft
Connections:
- no-connect marks 0 -> 2
Changed lines of the file:
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@@
 		(color 0 0 0 0)
+	)
+	(no_connect
+		(at 116.84 143.51)
+	)
+	(no_connect
+		(at 116.84 168.91)
 	)
 	(bus_entry

Commit message: better 15V GND
Connections:
- no-connect marks 2 -> 6
Changed lines of the file:
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@@
 	(title_block
 		(title "G6 Teensy 10-14 Arena")
-		(date "2026-08-03")
+		(date "2026-10-25")
 		(rev "v1.0")
 		(company "Reiser Lab @ Janelia | HHMI")
@@
 	)
 	(junction
-		(at 228.6 209.55)
-		(diameter 0)
-		(color 0 0 0 0)
-	)
-	(junction
 		(at 87.63 209.55)
 		(diameter 0)
@@
 	)
 	(no_connect
+		(at 116.84 118.11)
+	)
+	(no_connect
+		(at 116.84 66.04)
+	)
+	(no_connect
 		(at 116.84 143.51)
 	)
 	(no_connect
+		(at 116.84 40.64)
+	)
+	(no_connect
+		(at 116.84 92.71)
+	)
+	(no_connect
 		(at 116.84 168.91)
 	)
@@
 		)
 		(stroke
-			(width 0)
-			(type default)
-		)
-	)
-	(wire
-		(pts
-			(xy 275.59 209.55) (xy 228.6 209.55)
-		)
-		(stroke
