File: arena_10-14/panel_column.kicad_sch (KiCad schematic)
At the start: 5 parts, among them J7 Conn_01x05, J8 Conn_01x05, P1 NA

Commit message: rotate teensy
Parts:
- F1: LCSC Part # C46422913 -> C118413
Changed lines of the file:
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@@
 			)
 		)
-		(property "LCSC Part #" "C46422913"
+		(property "LCSC Part #" "C118413"
 			(at 154.94 50.8 0)
 			(hide yes)

Commit message: first moat
Parts:
- F1: LCSC Part # C118413 -> C126818
Changed lines of the file:
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@@
 			)
 		)
-		(property "LCSC Part #" "C118413"
+		(property "LCSC Part #" "C126818"
 			(at 154.94 50.8 0)
 			(hide yes)
@@
 			(project "arena_10-14"
 				(path "/056666d2-2c8f-491c-bcad-db3c517779a8/3aea6610-f2a3-4b21-99b1-2866223bb12f/22e744c9-b090-495f-8a7a-6f172c4fef79"
-					(reference "F11")
+					(reference "F6")
 					(unit 1)
 				)
 				(path "/056666d2-2c8f-491c-bcad-db3c517779a8/3aea6610-f2a3-4b21-99b1-2866223bb12f/2d48c774-5bc7-44a4-9df6-3d6978bb1a97"
-					(reference "F8")
+					(reference "F9")
 					(unit 1)
 				)
@@
 				)
 				(path "/056666d2-2c8f-491c-bcad-db3c517779a8/3aea6610-f2a3-4b21-99b1-2866223bb12f/5b4b3792-1e39-479f-bd98-38e020ce3fcb"
-					(reference "F9")
+					(reference "F10")
 					(unit 1)
 				)
 				(path "/056666d2-2c8f-491c-bcad-db3c517779a8/3aea6610-f2a3-4b21-99b1-2866223bb12f/92c2be2f-8271-448b-8aa4-e4b8407efff6"
-					(reference "F6")
+					(reference "F7")
 					(unit 1)
 				)
@@
 				)
 				(path "/056666d2-2c8f-491c-bcad-db3c517779a8/3aea6610-f2a3-4b21-99b1-2866223bb12f/f30e8937-4e73-4e94-bb30-d8448d44cc0d"
-					(reference "F7")
+					(reference "F8")
 					(unit 1)
 				)

Commit message: better 15V GND
Parts:
- F1: value 1206L005/110WR -> 1.1A PTC
Changed lines of the file:
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@@
 	(title_block
 		(title "G6 Teensy 10-14 Arena")
-		(date "2026-08-03")
+		(date "2026-10-25")
 		(rev "v1.0")
 		(company "Reiser Lab @ Janelia | HHMI")
@@
 			)
 		)
-		(property "Value" "1206L005/110WR"
+		(property "Value" "1.1A PTC"
 			(at 157.48 52.0699 0)
 			(show_name no)
