File: arena_10-14/power.kicad_sch (KiCad schematic)
At the start: 4 parts, among them J27 Barrel_Jack, J28 Barrel_Jack, SW1 SW_SPDT, U82 RB-0515D

Commit message: add jst and XT30, move DIO
Parts:
- removed J28: Barrel_Jack, arena_custom:DC-053D-20A, symbol Connector:Barrel_Jack
- added J35: JST PH, Connector_JST:JST_PH_B2B-PH-K_1x02_P2.00mm_Vertical, symbol Connector_Generic:Conn_01x02
- added J5: XT30, Connector_AMASS:AMASS_XT30UPB-F_1x02_P5.0mm_Vertical, symbol Connector_Generic:Conn_01x02
Connections:
- net +5V: now also J35.1 (Pin_1), J5.1 (Pin_1)
- net GND: now also J35.2 (Pin_2), J5.2 (Pin_2)

Commit message: first moat
Connections:
- net +5V: now also J5.2 (Pin_2); no longer J5.1 (Pin_1)
- net GND: now also J5.1 (Pin_1); no longer J5.2 (Pin_2)
Changed lines of the file:
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@@
 	(symbol
 		(lib_id "Connector_Generic:Conn_01x02")
-		(at 88.9 91.44 0)
+		(at 88.9 93.98 0)
+		(mirror x)
 		(unit 1)
 		(body_style 1)
@@
 		(fields_autoplaced yes)
 		(property "Reference" "J5"
-			(at 91.44 91.4399 0)
+			(at 91.44 93.9801 0)
 			(show_name no)
 			(do_not_autoplace no)
@@
 		)
 		(property "Value" "XT30"
-			(at 91.44 93.9799 0)
+			(at 91.44 91.4401 0)
 			(show_name no)
 			(do_not_autoplace no)
@@
 		)
 		(property "Footprint" "Connector_AMASS:AMASS_XT30UPB-F_1x02_P5.0mm_Vertical"
-			(at 88.9 91.44 0)
+			(at 88.9 93.98 0)
 			(hide yes)
 			(show_name no)
@@
 		)
 		(property "Datasheet" ""
-			(at 88.9 91.44 0)
+			(at 88.9 93.98 0)
 			(hide yes)
 			(show_name no)
@@
 		)
 		(property "Description" "Generic connector, single row, 01x02, script generated (kicad-library-utils/schlib/autogen/connector/)"
-			(at 88.9 91.44 0)
+			(at 88.9 93.98 0)
 			(hide yes)
 			(show_name no)
@@
 		)
 		(property "LCSC Part #" "C108769"
-			(at 88.9 91.44 0)
+			(at 88.9 93.98 0)
 			(hide yes)
 			(show_name no)

Commit message: Link DIO 3 & 4 DIR, place connectors
Parts:
- SW1: LCSC Part # C19189125 -> C2884789
Changed lines of the file:
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@@
 			)
 		)
-		(property "LCSC Part #" "C19189125"
+		(property "LCSC Part #" "C2884789"
 			(at 44.45 31.75 0)
 			(hide yes)
