File: arena_10-14/teensy.kicad_sch (KiCad schematic)
At the start: 36 parts, among them J1 Cetus RJ45 Magjack, J2 Qwiic, J28 Conn_01x24_Socket, J3 Conn_01x02, J36 Conn_01x24_Socket, J4 Conn_01x02, U1 Teensy4.1

Commit message: fix DIO labels
Parts:
- J28, J36: footprint PinSocket_1x24_P2.54mm_Vertical -> Connector_PinSocket_2.54mm:PinSocket_1x24_P2.54mm_Vertical
Connections:
- net +3.3V: no longer J28.15 (Pin_15), J36.3 (Pin_3)
- net AIN.A0: no longer J36.13 (Pin_13)
- net AIN.A1: no longer J36.12 (Pin_12)
- net D29_0_3V3: no longer J36.20 (Pin_20)
- net D35_0_3V3: no longer J36.22 (Pin_22)
- net DIO1/DIR: no longer J36.21 (Pin_21)
- net DIO2/DIR: no longer J36.23 (Pin_23)
- net DIO3/A: no longer J36.16 (Pin_16)
- net DIO3/DIR: no longer J36.17 (Pin_17)
- net DIO4/A: no longer J36.18 (Pin_18)
- net GND: now also U1.64 (GND); no longer J28.1 (Pin_1), J36.15 (Pin_15), J36.2 (Pin_2)
- net I2C.SCL: no longer J36.8 (Pin_8)
- net I2C.SDA: no longer J36.9 (Pin_9)
- net Qwiic_SCL: no longer J36.11 (Pin_11)
- net Qwiic_SDA: no longer J36.10 (Pin_10)
- net TNY.CIPO_B0: no longer J28.14 (Pin_14)
- net TNY.CIPO_B1: no longer J28.3 (Pin_3)
- net VIN: no longer J36.1 (Pin_1)
- net at R21.2, U1.45 (23_A9_CRX1_MCLK1): no longer J36.4 (Pin_4)
- net at R2.2, U1.4 (2_OUT2): no longer J28.4 (Pin_4)
- net at R3.2, U1.5 (3_LRCLK2): no longer J28.5 (Pin_5)
- net at R10.2, U1.12 (10_CS_MQSR): no longer J28.12 (Pin_12)
- net at R19.2, U1.23 (31_CTX3): no longer J28.23 (Pin_23)
- net at R23.2, U1.43 (21_A7_RX5_BCLK1): no longer J36.6 (Pin_6)
- net at R24.2, U1.35 (13_SCK_LED): no longer J36.14 (Pin_14)
- net at U1.30 (38_CS1_IN1): no longer J36.19 (Pin_19)
- net at R29.2, U1.25 (33_MCLK2): no longer J36.24 (Pin_24)
- net at R22.2, U1.44 (22_A8_CTX1): no longer J36.5 (Pin_5)
- net at U1.42 (20_A6_TX5_LRCLK1): no longer J36.7 (Pin_7)
- net at R16.2, U1.20 (28_RX7): no longer J28.20 (Pin_20)
- net at R8.2, U1.10 (8_TX2_IN1): no longer J28.10 (Pin_10)
- net at R6.2, U1.8 (6_OUT1D): no longer J28.8 (Pin_8)
- net at R14.2, U1.18 (26_A12_MOSI1): no longer J28.18 (Pin_18)
- net at R11.2, U1.13 (11_MOSI_CTX1): no longer J28.13 (Pin_13)
- net at R4.2, U1.6 (4_BCLK2): no longer J28.6 (Pin_6)
- net at R15.2, U1.19 (27_A13_SCK1): no longer J28.19 (Pin_19)
- net at R7.2, U1.9 (7_RX2_OUT1A): no longer J28.9 (Pin_9)
- net at R18.2, U1.22 (30_CRX3): no longer J28.22 (Pin_22)
- net at R12.2, U1.16 (24_A10_TX6_SCL2): no longer J28.16 (Pin_16)
- net at R9.2, U1.11 (9_OUT1C): no longer J28.11 (Pin_11)
- net at R13.2, U1.17 (25_A11_RX6_SDA2): no longer J28.17 (Pin_17)
- net at R1.2, U1.2 (0_RX1_CRX2_CS1): no longer J28.2 (Pin_2)
- net at R17.2, U1.21 (29_TX7): no longer J28.21 (Pin_21)
- net at R20.2, U1.24 (32_OUT1B): no longer J28.24 (Pin_24)
- net at R5.2, U1.7 (5_IN2): no longer J28.7 (Pin_7)
Other:
- note added: "Teensy Connectors"

Commit message: mount points near qwiic etc
Parts:
- J2: symbol Connector_Generic:Conn_01x04 -> Connector_Generic_MountingPin:Conn_01x04_MountingPin
Connections:
- net GND: now also J2.MP (MountPin)
